File: HandPICd32.kicad_pcb (KiCad board)
At the start: 4 copper layers, 100 x 100 mm, 334 parts, among them J1 Mini-DIN-6, J10 Conn-01x06, J11 Conn_02x03_Odd_Even, J12 Conn_01x06, J13 Conn_01x02, J2 DE9_Plug, J3 Conn_01x03, J4 DE15_Receptacle_HighDensity, J5 USB_B, J6 USB_A, J7 DE9_Plug, J8 AudioJack3, J9 Conn_01x06, SW1 SW_SPDT, SW2 SW_Push, U1 PIC32MZ2048EFH144T-I/PH, U2 74HCT273, U4 LM1117T-3.3, Y1 Crystal

Commit message: Add files via upload
Parts:
- U1: value PIC32MZ2048EFH144T-I/PH -> PIC32MZ2048EFH144-I/PH; footprint HandPICd32:TQFP144_PH_MCH-M -> HandPICd32:LQFP-144_20x20mm_P0.5mm-CUSTOM
- moved R11 19.4 mm to (127.2, 93.7), turned to 90 degrees
- moved C13 9.19 mm to (113.0, 81.2), turned to 180 degrees
- moved Y1 5.15 mm to (117.5, 88.2), turned to 90 degrees
- moved C12 4.95 mm to (113.0, 85.0), turned to 180 degrees
- moved C8 3.05 mm to (91.8, 82.5)
- moved C3 2.92 mm to (107.2, 117.5)
- moved C1 2.80 mm to (117.5, 106.8)
- moved C5 2.69 mm to (117.5, 95.2)
- moved C6 2.69 mm to (82.5, 105.2)
- moved C10 2.61 mm to (107.0, 82.5)
- moved C7 2.55 mm to (82.5, 97.8)
- moved C9 2.51 mm to (101.2, 82.5)
- moved C2 2.50 mm to (99.8, 117.5)
- moved C4 2.50 mm to (117.5, 99.8)
- moved C11 1.50 mm to (82.2, 115.5)
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- renumbered G102 to G104
Routing:
- net Pin24: track 113.0 -> 180.9 mm
- net Pin23: track 104.6 -> 164.1 mm, vias 2 -> 0
- net Pin113: track 138.0 -> 181.1 mm
- net Pin118: track 45.0 -> 74.7 mm, vias 0 -> 2
- net Pin104: track 75.3 -> 98.2 mm, vias 3 -> 4
- net Pin133: track 77.6 -> 100.0 mm
- net Pin69: track 136.2 -> 149.5 mm
- net /Pin44: track 20.1 -> 33.0 mm
- net Pin72: track 13.9 -> 26.2 mm
- net +5V: track 362.5 -> 350.7 mm
- net Pin28: track 89.5 -> 77.7 mm, vias 1 -> 2
- net Pin97: track 172.3 -> 183.3 mm, vias 1 -> 3
- net Pin30: track 98.4 -> 108.3 mm
- net Pin20: track 120.2 -> 129.3 mm, vias 2 -> 1
- net /Pin16: track 23.0 -> 14.4 mm, vias 1 -> 0
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Other:
- board text added: "Professor Steven Chad Burrow stevenchadburrow@gmail.com github.com/stevenchadburrow youtube.com/user/stevenchadburrow Nov 2024"
- board text removed: "Professor Steven Chad Burrow stevenchadburrow@gmail.com github.com/stevenchadburrow youtube.com/user/stevenchadburrow Oct 2024"

Commit message: Add files via upload
Parts:
- removed C15, C17: C_Polarized_Small_US, Capacitor_THT:CP_Radial_D6.3mm_P2.50mm
- removed C18: C_Small, Capacitor_THT:C_Disc_D3.0mm_W1.6mm_P2.50mm
- removed J10: Conn-01x06, Connector_PinSocket_2.54mm:PinSocket_1x06_P2.54mm_Horizontal
- removed J13: Conn_01x02, Connector_PinHeader_2.54mm:PinHeader_1x02_P2.54mm_Vertical
- removed J3: Conn_01x03, Connector_PinHeader_2.54mm:PinHeader_1x03_P2.54mm_Vertical
- removed TP100, TP101, TP102, TP104, TP109, TP110, TP111, TP112, TP113, TP114, TP116, TP121, TP128, TP129, TP131, TP138, TP139, TP27, TP29, TP31, TP32, TP33, TP34, TP35, TP41, TP42, TP43, TP48, TP49, TP56, TP57, TP59, TP60, TP61, TP62, TP63, TP64, TP66, TP67, TP68, TP69, TP70, TP71, TP75, TP76, TP77, TP78, TP79, TP82, TP83, TP84, TP85, TP86, TP87, TP88, TP92, TP93, TP94, TP95, TP96, TP97, TP98, TP99: TestPoint, HandPICd32:TestPointStdTHT
- removed U2: 74HCT273, Package_DIP:DIP-20_W7.62mm_Socket
- added C24: C_Polarized_Small_US, Capacitor_THT:CP_Radial_D6.3mm_P2.50mm, F.Cu at (87.5, 82.5)
- added J14: Conn_02x02_Odd_Even, Connector_PinHeader_2.54mm:PinHeader_2x02_P2.54mm_Vertical, F.Cu at (115.0, 115.0)
- added R20: R_US, Resistor_THT:R_Axial_DIN0204_L3.6mm_D1.6mm_P7.62mm_Horizontal, F.Cu at (67.1, 115.0)
- added R21: R_US, Resistor_THT:R_Axial_DIN0204_L3.6mm_D1.6mm_P7.62mm_Horizontal, F.Cu at (67.1, 112.5)
- added R23: R_US, Resistor_THT:R_Axial_DIN0204_L3.6mm_D1.6mm_P7.62mm_Horizontal, F.Cu at (67.1, 110.0)
- added R24: R_US, Resistor_THT:R_Axial_DIN0204_L3.6mm_D1.6mm_P7.62mm_Horizontal, F.Cu at (67.1, 107.5)
- added R25: R_US, Resistor_THT:R_Axial_DIN0204_L3.6mm_D1.6mm_P7.62mm_Horizontal, F.Cu at (67.1, 105.0)
- added R26: R_US, Resistor_THT:R_Axial_DIN0204_L3.6mm_D1.6mm_P7.62mm_Horizontal, F.Cu at (67.1, 102.5)
- added R27: R_US, Resistor_THT:R_Axial_DIN0204_L3.6mm_D1.6mm_P7.62mm_Horizontal, F.Cu at (67.1, 100.0)
- added R28: R_US, Resistor_THT:R_Axial_DIN0204_L3.6mm_D1.6mm_P7.62mm_Horizontal, F.Cu at (67.1, 97.5)
- added R29: R_US, Resistor_THT:R_Axial_DIN0204_L3.6mm_D1.6mm_P7.62mm_Horizontal, F.Cu at (67.1, 95.0)
- added R30: R_US, Resistor_THT:R_Axial_DIN0204_L3.6mm_D1.6mm_P7.62mm_Horizontal, F.Cu at (67.1, 92.5)
- added R31: R_US, Resistor_THT:R_Axial_DIN0204_L3.6mm_D1.6mm_P7.62mm_Horizontal, F.Cu at (67.1, 90.0)
- added R32: R_US, Resistor_THT:R_Axial_DIN0204_L3.6mm_D1.6mm_P7.62mm_Horizontal, F.Cu at (67.1, 87.5)
- added R33: R_US, Resistor_THT:R_Axial_DIN0204_L3.6mm_D1.6mm_P7.62mm_Horizontal, F.Cu at (67.1, 85.0)
- added R34: R_US, Resistor_THT:R_Axial_DIN0204_L3.6mm_D1.6mm_P7.62mm_Horizontal, F.Cu at (67.1, 82.5)
- added R35: R_US, Resistor_THT:R_Axial_DIN0204_L3.6mm_D1.6mm_P7.62mm_Horizontal, F.Cu at (67.1, 80.0)
- added R36: R_US, Resistor_THT:R_Axial_DIN0204_L3.6mm_D1.6mm_P7.62mm_Horizontal, F.Cu at (59.5, 117.5)
- added R37: R_US, Resistor_THT:R_Axial_DIN0204_L3.6mm_D1.6mm_P7.62mm_Horizontal, F.Cu at (110.0, 70.8)
- added R38: R_US, Resistor_THT:R_Axial_DIN0204_L3.6mm_D1.6mm_P7.62mm_Horizontal, F.Cu at (77.6, 107.5)
- added R39: R_US, Resistor_THT:R_Axial_DIN0204_L3.6mm_D1.6mm_P7.62mm_Horizontal, F.Cu at (77.6, 105.0)
- added R40: R_US, Resistor_THT:R_Axial_DIN0204_L3.6mm_D1.6mm_P7.62mm_Horizontal, F.Cu at (77.6, 102.5)
- added R41: R_US, Resistor_THT:R_Axial_DIN0204_L3.6mm_D1.6mm_P7.62mm_Horizontal, F.Cu at (77.6, 100.0)
- added R42: R_US, Resistor_THT:R_Axial_DIN0204_L3.6mm_D1.6mm_P7.62mm_Horizontal, F.Cu at (77.6, 97.5)
- added R43: R_US, Resistor_THT:R_Axial_DIN0204_L3.6mm_D1.6mm_P7.62mm_Horizontal, F.Cu at (77.6, 95.0)
- added R44: R_US, Resistor_THT:R_Axial_DIN0204_L3.6mm_D1.6mm_P7.62mm_Horizontal, F.Cu at (77.6, 92.5)
- added R45: R_US, Resistor_THT:R_Axial_DIN0204_L3.6mm_D1.6mm_P7.62mm_Horizontal, F.Cu at (77.6, 90.0)
- added R46: R_US, Resistor_THT:R_Axial_DIN0204_L3.6mm_D1.6mm_P7.62mm_Horizontal, F.Cu at (77.6, 87.5)
- added R47: R_US, Resistor_THT:R_Axial_DIN0204_L3.6mm_D1.6mm_P7.62mm_Horizontal, F.Cu at (77.6, 85.0)
- added R48: R_US, Resistor_THT:R_Axial_DIN0204_L3.6mm_D1.6mm_P7.62mm_Horizontal, F.Cu at (77.6, 82.5)
- added R49: R_US, Resistor_THT:R_Axial_DIN0204_L3.6mm_D1.6mm_P7.62mm_Horizontal, F.Cu at (77.6, 80.0)
- added R50: R_US, Resistor_THT:R_Axial_DIN0204_L3.6mm_D1.6mm_P7.62mm_Horizontal, F.Cu at (110.0, 73.2)
- added R51: R_US, Resistor_THT:R_Axial_DIN0207_L6.3mm_D2.5mm_P10.16mm_Horizontal, F.Cu at (82.9, 73.0)
- added R52: R_US, Resistor_THT:R_Axial_DIN0207_L6.3mm_D2.5mm_P10.16mm_Horizontal, F.Cu at (82.9, 69.5)
- added R53: R_US, Resistor_THT:R_Axial_DIN0207_L6.3mm_D2.5mm_P10.16mm_Horizontal, F.Cu at (103.8, 66.8)
- added R54: R_US, Resistor_THT:R_Axial_DIN0207_L6.3mm_D2.5mm_P10.16mm_Horizontal, F.Cu at (100.2, 66.8)
- added R55: R_US, Resistor_THT:R_Axial_DIN0207_L6.3mm_D2.5mm_P10.16mm_Horizontal, F.Cu at (96.8, 66.8)
- added R56: R_US, Resistor_THT:R_Axial_DIN0207_L6.3mm_D2.5mm_P10.16mm_Horizontal, F.Cu at (69.7, 76.5)
- added R57: R_US, Resistor_THT:R_Axial_DIN0207_L6.3mm_D2.5mm_P10.16mm_Horizontal, F.Cu at (69.7, 73.0)
- added R58: R_US, Resistor_THT:R_Axial_DIN0207_L6.3mm_D2.5mm_P10.16mm_Horizontal, F.Cu at (82.9, 76.5)
- added SW3: SW_Push, Button_Switch_THT:SW_Tactile_SPST_Angled_PTS645Vx83-2LFS, F.Cu at (147.0, 62.0)
- J11: value Conn_02x03_Odd_Even -> Micro_SD_Card; footprint Connector_PinHeader_2.54mm:PinHeader_2x03_P2.54mm_Vertical -> Connector_Card:microSD_HC_Hirose_DM3D-SF
- R12, R13, R14, R15: footprint Resistor_THT:R_Axial_DIN0207_L6.3mm_D2.5mm_P10.16mm_Horizontal -> Resistor_THT:R_Axial_DIN0204_L3.6mm_D1.6mm_P7.62mm_Horizontal
- moved J1 91.4 mm to (54.3, 132.0), turned to 90 degrees
- moved C19 74.5 mm to (63.0, 131.0), turned to 90 degrees
- moved J11 66.4 mm to (142.3, 130.5), turned to 90 degrees
- moved R18 61.8 mm to (122.8, 70.5), turned to -90 degrees
- moved TP9 57.3 mm to (145.7, 139.0), turned to 0 degrees
- moved R2 55.7 mm to (76.2, 128.0), turned to 180 degrees
- moved TP8 54.1 mm to (140.6, 139.0), turned to 0 degrees
- moved R13 52.7 mm to (77.6, 115.0), turned to 180 degrees
- moved TP7 50.1 mm to (121.5, 83.8), turned to 180 degrees
- moved TP132 46.3 mm to (121.5, 86.3), turned to -90 degrees
- moved TP137 46.3 mm to (124.0, 83.8)
- moved TP58 46.3 mm to (124.0, 86.3)
- moved R12 45.6 mm to (70.0, 117.5), turned to 0 degrees
- moved TP91 45.0 mm to (124.0, 88.8)
- moved TP89 43.4 mm to (124.0, 91.4)
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Connections:
- net /Pin78 renamed Pin78
- net Pin135 renamed /Pin135
- net Pin138 renamed /Pin138
- net Pin142 renamed /Pin142
- net Pin143 renamed /Pin143
- net Pin144 renamed /Pin144
- net Pin23 renamed /Pin23
- net Pin3 renamed /Pin3
- net Pin4 renamed /Pin4
- net Pin5 renamed /Pin5
- C16 pad 1: Pin24 -> Net-(C16-Pad1)
- C16 pad 2: AUDIO-NEG-B -> AUDIO-OUT-RIGHT
- D1 pad 2: +5V -> +3V3
- J11 pad 1: USB-A-D+ -> unconnected-(J11-DAT2-Pad1)
- J11 pad 2: USB-A-D- -> Pin118
- J11 pad 3: Pin77 -> Pin121
- J11 pad 4: Pin76 -> +3V3
- J11 pad 5: USB-B-D+ -> Pin109
- J11 pad 6: USB-B-D- -> GND
- J2 pad 1: Pin114 -> Pin19
- J2 pad 2: Pin115 -> Pin51
- J2 pad 3: Pin116 -> Pin52
- J2 pad 4: Pin117 -> Pin53
- J2 pad 6: Pin131 -> Pin92
- J2 pad 7: Pin30 -> Pin94
- J2 pad 9: Pin132 -> Pin93
- J6 pad 2: USB-A-D- -> Pin76
- J6 pad 3: USB-A-D+ -> Pin77
- J7 pad 1: Pin133 -> Pin124
- J7 pad 2: Pin134 -> Pin125
- J7 pad 3: Pin10 -> Pin79
- J7 pad 4: Pin9 -> Pin90
- J7 pad 6: Pin28 -> Pin91
- J7 pad 7: Pin30 -> Pin94
- J7 pad 9: Pin29 -> Pin80
- J8 pad R: AUDIO-OUT -> AUDIO-OUT-RIGHT
- J8 pad T: AUDIO-OUT -> AUDIO-OUT-LEFT
- R10 pad 2: RED-A -> Pin103
- R12 pad 1: GND -> Net-(R12-Pad1)
- R12 pad 2: AUDIO-OUT -> GND
- R13 pad 1: AUDIO-OUT -> Pin7
- R13 pad 2: AUDIO-COMBINED -> Net-(R12-Pad1)
- R14 pad 1: AUDIO-COMBINED -> Net-(R14-Pad1)
- R14 pad 2: AUDIO-NEG-B -> Net-(R12-Pad1)
- R15 pad 1: AUDIO-COMBINED -> Pin8
- R15 pad 2: AUDIO-NEG-A -> Net-(R14-Pad1)
- R16 pad 1: Pin30 -> Pin94
- R18 pad 1: Pin27 -> Pin126
- R2 pad 2: SPI-POWER -> +3V3
- R3 pad 2: BLUE-B -> Pin81
- R4 pad 2: BLUE-A -> Pin82
- R5 pad 2: GREEN-C -> Pin83
- R6 pad 2: GREEN-B -> Pin84
- R7 pad 2: GREEN-A -> Pin100
- R8 pad 2: RED-C -> Pin101
- R9 pad 2: RED-B -> Pin102
- RN1 pad 2: Pin10 -> Pin124
- RN1 pad 3: Pin9 -> Pin125
- RN1 pad 4: Pin28 -> Pin79
- RN1 pad 5: Pin29 -> Pin90
- RN1 pad 6: Pin97 -> Pin91
- RN1 pad 7: Pin98 -> Pin80
- RN2 pad 2: Pin114 -> Pin19
- RN2 pad 3: Pin115 -> Pin51
- RN2 pad 4: Pin116 -> Pin52
- RN2 pad 5: Pin117 -> Pin53
- RN2 pad 6: Pin131 -> Pin92
- RN2 pad 7: Pin132 -> Pin93
- RN2 pad 8: Pin133 -> Pin97
- RN2 pad 9: Pin134 -> Pin98
- TP20 pad 1: Pin24 -> /Pin24
- TP23 pad 1: Pin27 -> Pin121
- TP24 pad 1: Pin28 -> Pin120
- TP25 pad 1: /Pin19 -> +3V3
- TP26 pad 1: Pin29 -> GND
- TP7 pad 1: /Pin7 -> +5V
- TP8 pad 1: /Pin8 -> Pin118
- TP9 pad 1: Pin9 -> Pin109
- U1 pad 100: /Pin100 -> Pin100
- U1 pad 101: /Pin101 -> Pin101
- U1 pad 102: /Pin102 -> Pin102
- U1 pad 103: /Pin103 -> Pin103
- U1 pad 124: /Pin124 -> Pin124
- U1 pad 125: /Pin125 -> Pin125
- U1 pad 126: /Pin126 -> Pin126
- U1 pad 19: /Pin19 -> Pin19
- U1 pad 24: Pin24 -> /Pin24
- U1 pad 43: /Pin43 -> Pin43
- U1 pad 44: /Pin44 -> Pin44
- U1 pad 45: /Pin45 -> Pin45
- U1 pad 46: /Pin46 -> Pin46
- U1 pad 51: /Pin51 -> Pin51
- U1 pad 52: /Pin52 -> Pin52
- U1 pad 53: /Pin53 -> Pin53
- U1 pad 65: /Pin65 -> Pin65
- U1 pad 66: /Pin66 -> Pin66
- U1 pad 67: /Pin67 -> Pin67
- U1 pad 68: /Pin68 -> Pin68
- U1 pad 7: /Pin7 -> Pin7
- U1 pad 79: /Pin79 -> Pin79
- U1 pad 8: /Pin8 -> Pin8
- U1 pad 80: /Pin80 -> Pin80
- U1 pad 81: /Pin81 -> Pin81
- U1 pad 82: /Pin82 -> Pin82
- U1 pad 83: /Pin83 -> Pin83
- U1 pad 84: /Pin84 -> Pin84
- U1 pad 90: /Pin90 -> Pin90
- U1 pad 91: /Pin91 -> Pin91
- U1 pad 92: /Pin92 -> Pin92
- U1 pad 93: /Pin93 -> Pin93
- U1 pad 94: /Pin94 -> Pin94
Routing:
- net Pin24: track 180.9 -> 0.00 mm, vias 2 -> 0
- net Pin93: track 0.00 -> 135.9 mm, vias 0 -> 3
- net /Pin23: track 164.1 -> 31.7 mm, vias 0 -> 2
- net Pin79: track 0.00 -> 126.6 mm, vias 0 -> 5
- net Pin94: track 0.00 -> 119.6 mm, vias 0 -> 3
- net Pin91: track 0.00 -> 113.3 mm, vias 0 -> 3
- net Pin92: track 0.00 -> 109.9 mm, vias 0 -> 1
- net Pin90: track 0.00 -> 98.3 mm, vias 0 -> 2
- net Pin53: track 0.00 -> 97.9 mm, vias 0 -> 3
- net Pin113: track 181.1 -> 83.6 mm, vias 2 -> 1
- net Pin80: track 0.00 -> 95.2 mm, vias 0 -> 2
- net USB-A-D+: track 88.5 -> 0.00 mm, vias 2 -> 0
- net Pin126: track 0.00 -> 87.7 mm, vias 0 -> 2
- net Pin27: track 128.9 -> 42.4 mm
- net Pin124: track 0.00 -> 85.0 mm, vias 0 -> 2
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Other:
- board text added: "*"
- board text added: "5V"
- board text added: "GND"
- board text added: "John 3:16 For God so loved the world, that he gave his only begotten Son, that whosoever believeth in him should not perish, but have everlasting life."
- board text added: "Professor Steven Chad Burrow stevenchadburrow@gmail.com github.com/stevenchadburrow youtube.com/user/stevenchadburrow Jan 2025"
- board text removed: "5V0"
- board text removed: "A"
- board text removed: "B"
- board text removed: "Professor Steven Chad Burrow stevenchadburrow@gmail.com github.com/stevenchadburrow youtube.com/user/stevenchadburrow Nov 2024"
