File: HandPICd32.kicad_sch (KiCad schematic)
At the start: 329 parts, among them J1 USB_B, J10 Conn-01x06, J11 Conn_02x03_Odd_Even, J12 Conn_01x06, J13 Conn_01x02, J3 Conn_01x03, J3 DE15_Receptacle_HighDensity, J3 USB_A, J5 Mini-DIN-6, J8 AudioJack3, J8 DE9_Plug, J9 Conn_01x06, SW1 SW_SPDT, SW2 SW_Push, U1 PIC32MZ2048EFH144T-I/PH, U2 74HCT273, U4 LM1117T-3.3, Y1 Crystal

Commit message: Add files via upload
Parts:
- U1: value PIC32MZ2048EFH144T-I/PH -> PIC32MZ2048EFH144-I/PH; footprint HandPICd32:TQFP144_PH_MCH-M -> HandPICd32:LQFP-144_20x20mm_P0.5mm-CUSTOM
Changed lines of the file:
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@@
       (effects (font (size 1.524 1.524)))
     )
-    (property "Value" "PIC32MZ2048EFH144T-I/PH" (at 99.06 17.78 0)
+    (property "Value" "PIC32MZ2048EFH144-I/PH" (at 99.06 17.78 0)
       (effects (font (size 1.524 1.524)))
     )
-    (property "Footprint" "HandPICd32:TQFP144_PH_MCH-M" (at 27.94 25.4 0)
+    (property "Footprint" "HandPICd32:LQFP-144_20x20mm_P0.5mm-CUSTOM" (at 27.94 25.4 0)
       (effects (font (size 1.27 1.27) italic) hide)
     )
-    (property "Datasheet" "PIC32MZ2048EFH144T-I/PH" (at 27.94 25.4 0)
+    (property "Datasheet" "PIC32MZ2048EFH144-I/PH" (at 27.94 25.4 0)
       (effects (font (size 1.27 1.27) italic) hide)
     )
@@
       (effects (font (size 1.524 1.524)))
     )
-    (property "Value" "PIC32MZ2048EFH144T-I/PH" (at 274.32 17.78 0)
+    (property "Value" "PIC32MZ2048EFH144-I/PH" (at 274.32 17.78 0)
       (effects (font (size 1.524 1.524)))
     )
-    (property "Footprint" "HandPICd32:TQFP144_PH_MCH-M" (at 203.2 25.4 0)
+    (property "Footprint" "HandPICd32:LQFP-144_20x20mm_P0.5mm-CUSTOM" (at 203.2 25.4 0)
       (effects (font (size 1.27 1.27) italic) hide)
     )
-    (property "Datasheet" "PIC32MZ2048EFH144T-I/PH" (at 203.2 25.4 0)
+    (property "Datasheet" "PIC32MZ2048EFH144-I/PH" (at 203.2 25.4 0)
       (effects (font (size 1.27 1.27) italic) hide)
     )

Commit message: Add files via upload
Parts:
- removed C15, C17: C_Polarized_Small_US, Capacitor_THT:CP_Radial_D6.3mm_P2.50mm, symbol Device:C_Polarized_Small_US
- removed C18: C_Small, Capacitor_THT:C_Disc_D3.0mm_W1.6mm_P2.50mm, symbol Device:C_Small
- removed J10: Conn-01x06, Connector_PinSocket_2.54mm:PinSocket_1x06_P2.54mm_Horizontal, symbol Connector_Generic:Conn_01x06
- removed J11: Conn_02x03_Odd_Even, Connector_PinHeader_2.54mm:PinHeader_2x03_P2.54mm_Vertical, symbol Connector_Generic:Conn_02x03_Odd_Even
- removed J13: Conn_01x02, Connector_PinHeader_2.54mm:PinHeader_1x02_P2.54mm_Vertical, symbol Connector_Generic:Conn_01x02
- removed J3: Conn_01x03, Connector_PinHeader_2.54mm:PinHeader_1x03_P2.54mm_Vertical, symbol Connector_Generic:Conn_01x03
- removed TP100, TP101, TP102, TP104, TP109, TP110, TP111, TP112, TP113, TP114, TP116, TP121, TP128, TP129, TP131, TP138, TP139, TP27, TP29, TP31, TP32, TP33, TP34, TP35, TP41, TP42, TP43, TP48, TP49, TP56, TP57, TP59, TP60, TP61, TP62, TP63, TP64, TP66, TP67, TP68, TP69, TP70, TP71, TP75, TP76, TP77, TP78, TP79, TP82, TP83, TP84, TP85, TP86, TP87, TP88, TP92, TP93, TP94, TP95, TP96, TP97, TP98, TP99: TestPoint, HandPICd32:TestPointStdTHT, symbol Connector:TestPoint
- removed U2: 74HCT273, Package_DIP:DIP-20_W7.62mm_Socket, symbol 74xx:74HCT273
- added C24: C_Polarized_Small_US, Capacitor_THT:CP_Radial_D6.3mm_P2.50mm, symbol Device:C_Polarized_Small_US
- added J11: Micro_SD_Card, Connector_Card:microSD_HC_Hirose_DM3D-SF, symbol Connector:Micro_SD_Card
- added J14: Conn_02x02_Odd_Even, Connector_PinHeader_2.54mm:PinHeader_2x02_P2.54mm_Vertical, symbol Connector_Generic:Conn_02x02_Odd_Even
- added R20, R21, R23, R24, R25, R26, R27, R28, R29, R30, R31, R32, R33, R34, R35, R36, R37, R38, R39, R40, R41, R42, R43, R44, R45, R46, R47, R48, R49, R50: R_US, Resistor_THT:R_Axial_DIN0204_L3.6mm_D1.6mm_P7.62mm_Horizontal, symbol Device:R_US
- added R51, R52, R53, R54, R55, R56, R57, R58: R_US, Resistor_THT:R_Axial_DIN0207_L6.3mm_D2.5mm_P10.16mm_Horizontal, symbol Device:R_US
- added SW3: SW_Push, Button_Switch_THT:SW_Tactile_SPST_Angled_PTS645Vx83-2LFS, symbol Switch:SW_Push
- R12, R13, R15: footprint Resistor_THT:R_Axial_DIN0207_L6.3mm_D2.5mm_P10.16mm_Horizontal -> Resistor_THT:R_Axial_DIN0204_L3.6mm_D1.6mm_P7.62mm_Horizontal; Field4 10k -> 20K
- R14: footprint Resistor_THT:R_Axial_DIN0207_L6.3mm_D2.5mm_P10.16mm_Horizontal -> Resistor_THT:R_Axial_DIN0204_L3.6mm_D1.6mm_P7.62mm_Horizontal; Field4 10k -> 10K
- R17: Field4 >220 ohms -> >100 ohms
Connections:
- net BLUE-A is gone; now on net Pin82: R4.2
- net BLUE-B is gone; now on net Pin81: R3.2
- net GREEN-A is gone; now on net Pin100: R7.2
- net GREEN-B is gone; now on net Pin84: R6.2
- net GREEN-C is gone; now on net Pin83: R5.2
- net RED-A is gone; now on net Pin103: R10.2
- net RED-B is gone; now on net Pin102: R9.2
- net RED-C is gone; now on net Pin101: R8.2
- net SPI-POWER is gone; now on net +3V3: R2.2
- net USB-A-D+ is gone; now on net Pin77: J3.3 (D+)
- net USB-A-D- is gone; now on net Pin76: J3.2 (D-)
- net +3V3: now also D1.2 (A), TP25.1, J11.4 (VDD)
- net +5V: now also TP7.1; no longer D1.2 (A)
- net BLUE: now also R51.1, R52.1, R58.1
- net GND: now also R12.2, TP26.1, J11.6 (VSS), J11.9 (SHIELD), R36.2, R37.2, R50.2, SW3.2; no longer R12.1
- net GREEN: now also R53.1, R54.1, R55.1
- net Pin10: now also R39.1; no longer J8.3, RN1.2 (R1)
- net Pin109: now also TP9.1, J11.5 (CLK)
- net Pin114: now also R20.1; no longer J8.1, RN2.2 (R1)
- net Pin115: now also R23.1; no longer J8.2, RN2.3 (R2)
- net Pin116: now also R25.1; no longer J8.3, RN2.4 (R3)
- net Pin117: now also R27.1; no longer J8.4, RN2.5 (R4)
- net Pin118: now also TP8.1, J11.2 (DAT3/CD)
- net Pin120: now also TP24.1, J11.7 (DAT0)
- net Pin121: now also TP23.1, J11.3 (CMD)
- net Pin124: now also J8.1, RN1.2 (R1)
- net Pin125: now also J8.2, RN1.3 (R2)
- net Pin126: now also R18.1, SW3.1
- net Pin131: now also R29.1; no longer J8.6, RN2.6 (R5)
- net Pin132: now also R31.1; no longer J8.9, RN2.7 (R6)
- net Pin133: now also R33.1; no longer J8.1, RN2.8 (R7)
- net Pin134: now also R35.1; no longer J8.2, RN2.9 (R8)
- net Pin19: now also J8.1, RN2.2 (R1); no longer TP25.1
- net Pin24: no longer C16.1
- net Pin27: now also R41.1; no longer R18.1, TP23.1
- net Pin28: now also R45.1; no longer J8.6, RN1.4 (R3), TP24.1
- net Pin29: now also R47.1; no longer J8.9, RN1.5 (R4), TP26.1
- net Pin30: now also R49.1; no longer J8.7, J8.7, R16.1
- net Pin43: now also R58.2
- net Pin44: now also R51.2
- net Pin45: now also R52.2
- net Pin46: now also R53.2
- net Pin51: now also J8.2, RN2.3 (R2)
- net Pin52: now also J8.3, RN2.4 (R3)
- net Pin53: now also J8.4, RN2.5 (R4)
- net Pin65: now also R54.2
- net Pin66: now also R55.2
- net Pin67: now also R56.2
- net Pin68: now also R57.2
- net Pin7: now also R13.1; no longer TP7.1
- net Pin76: now also J14.2 (Pin_2)
- net Pin77: now also J14.1 (Pin_1)
- net Pin79: now also J8.3, RN1.4 (R3)
- net Pin8: now also R15.1; no longer TP8.1
- net Pin80: now also J8.9, RN1.7 (R6)
- net Pin9: now also R43.1; no longer J8.4, RN1.3 (R2), TP9.1
- net Pin90: now also J8.4, RN1.5 (R4)
- net Pin91: now also J8.6, RN1.6 (R5)
- net Pin92: now also J8.6, RN2.6 (R5)
- net Pin93: now also J8.9, RN2.7 (R6)
- net Pin94: now also J8.7, J8.7, R16.1
- net Pin97: now also RN2.8 (R7); no longer RN1.6 (R5)
- net Pin98: now also RN2.9 (R8); no longer RN1.7 (R6)
- net RED: now also R56.1, R57.1
- net USB-B-D+: now also J14.3 (Pin_3)
- net USB-B-D-: now also J14.4 (Pin_4)
- removed net AUDIO-COMBINED: R13.2, R14.1, R15.1
- net AUDIO-NEG-A: no longer names the net of R15.2
- net AUDIO-NEG-A: now also R14.1, R38.2
- net AUDIO-NEG-B: no longer names the net of R14.2
- net AUDIO-NEG-B: now also R12.1, R13.2; no longer C16.2
- removed net AUDIO-OUT: J8.R, J8.T, R12.2, R13.1
- new net: R20.2, R21.2, R36.1
- new net: C24.1, R34.1, R35.2
- new net: R40.1, R41.2, R42.2
- new net: R38.1, R39.2, R40.2
- new net: R21.1, R23.2, R24.2
- new net: R26.1, R27.2, R28.2
- new net: R24.1, R25.2, R26.2
- new net: R46.1, R47.2, R48.2
- new net: R44.1, R45.2, R46.2
- new net: C16.1, R48.1, R49.2
- new net: R42.1, R43.2, R44.2
- new net: R32.1, R33.2, R34.2
- new net: R28.1, R29.2, R30.2
- new net: R30.1, R31.2, R32.2
- new net AUDIO-OUT-LEFT: C24.2, J8.T, R37.1
- new net AUDIO-OUT-RIGHT: C16.2, J8.R, R50.1
- no-connect marks 138 -> 140
Other:
- note added: "// Video Color Signals PORTH // Video Clock Signals Pin104,RD0,PIXEL-CLOCK Pin119,RD5,VISIBLE-CLOCK Pin110,RD2,H-SYNC Pin111,RD3,V-SYNC // Audio PORTJ // SDcard Pin120,RD6,MISO Pin121,RD7,MOSI Pin109,RD1,SCK1 Pin118,RD4,CS // PS/2 Keyboard/Mouse Pin98,RD10,KEY-CLK Pin99,RD11,KEY-DAT Pin112,RD12,MOUSE-CLK Pin113,RD13,MOUSE-DAT // Joysticks Pin19,RK0,JOY-A-UP Pin51,RK1,JOY-A-DOWN Pin52,RK2,JOY-A-LE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"
- note added: "High Byte of PORTH RGB-332 Low Byte of PORTH RGB-233 Ohms: Red 510, 910, 2000, 3300, 6200 Green 510, 910, 2000, 3900, 7500, 15000 Blue 430, 820, 3900, 7500, 15000"
- note added: "If only using 6-bit, then resistors must be 1% is ok I believe. If using 8-bit, then something like 0.25% is needed."
- note added: "PIXEL-CLOCK"
- note added: "Test Points for SDcard"
- note added: "USBID"
- note added: "VISIBLE-CLOCK"
- note added: "https://falstad.com/circuit/circuitjs.html?ctz=CQAgjCAMB0l3BWcMBMcUHYMGZIA4UA2ATmIxAUgpABZsKBTAWjDACgAlcQ8DHsHsR5UqNKtmj0RUaAjYBlXv2IoQQ8CqjgQAMwCGAGwDODLSgVKQKMWp7XpEfcdNVzisHyt48trz6qOhiZmFh482NiC4ZFagc4h7p7YeDS+yakBukEuVqGedKrqBbFZ8a55PDR4VEXVJU7B5Yk8CCg+6q3+2g055gDu3JbqYVBsA9iqaO12+KMDApYLKNZzg8up6uurSytLGKqQY2v7vpgHR3uqCxMiF+FoaQ+H8-cB4YT+dyCR098f2+8fAsaAtnoMQVFaKCvhDwYQMjD4b4aEiwcCkQsEGBzi8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"
- note removed: "// Video Color Signals Pin5,RE7,RED-A Pin4,RE6,RED-B Pin3,RE5,RED-C Pin144,RE4,GREEN-A Pin143,RE3,GREEN-B Pin142,RE2,GREEN-C Pin138,RE1,BLUE-A Pin135,RE0,BLUE-B // Video Clock Signals Pin104,RD0,PIXEL-CLOCK Pin119,RD5,VISIBLE-CLOCK Pin110,RD2,H-SYNC Pin111,RD3,V-SYNC // Audio Pin23,RE8,AUDIO-A Pin24,RE9,AUDIO-B // SPI SDcard Adapter Pin120,RD6,MISO Pin121,RD7,MOSI Pin109,RD1,SCK1 Pin118,RD4,CS //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"
- note removed: "Micro SD Card Adapter"
- note removed: "Red/Green-A = 820 ohms Red/Green-B = 1600 ohms Red/Green-C = 3300 ohms Blue-A = 680 ohms Blue-B = 1500 ohms"
